Commit message: Fix the camera

File: tel_map/urdf/sakura.urdf.xacro (robot description, xacro)
@@ -26,7 +26,7 @@
       <origin xyz="0 0 0" rpy="0 0 0"/>
       <mass value="200.0"/>
-      <inertia ixx="0.1" ixy="-0.001" ixz="0.0001"
-               iyy="0.1" iyz="0.001"
-               izz="0.1" />
+      <inertia ixx="0.15" ixy="0.001" ixz="0.001"
+               iyy="0.15" iyz="0.001"
+               izz="0.15" />
     </inertial>
   </link>
@@ -338,9 +338,9 @@
     </visual>
     <inertial>
-      <mass value="0.114" />
+      <mass value="0.100" />
       <origin xyz="-0.0 0.0 0.0" rpy="0 0 0"/>
-      <inertia ixx="0.001" ixy="0.0" ixz="0.0"
-               iyy="0.001" iyz="0.0"
-               izz="0.001" />
+      <inertia ixx="0.000001" ixy="0.0001" ixz="0.0001"
+               iyy="0.000001" iyz="0.0001"
+               izz="0.000001" />
     </inertial>
   </link>
@@ -530,5 +530,5 @@
       <inertial>
       <origin xyz="0 0 0.02" rpy="0 0 0"/>
-      <mass value="0.001" />
+      <mass value="0.0001" />
       <inertia  ixx="0.0" ixy="0.0"  ixz="0.0"  iyy="0.0"  iyz="0.0"  izz="0.0" />
       </inertial>
@@ -556,5 +556,5 @@
       <inertial>
       <origin xyz="0 0 0.02" rpy="0 0 0"/>
-      <mass value="0.001" />
+      <mass value="0.0001" />
       <inertia  ixx="0.0" ixy="0.0"  ixz="0.0"  iyy="0.0"  iyz="0.0"  izz="0.0" />
       </inertial>

Commit message: Fix the gripper

File: tel_map/urdf/sakura.urdf.xacro (robot description, xacro)
@@ -524,12 +524,12 @@
       <parent link="hand"/>
       <child link="finger1"/>
-      <limit lower="0.0" upper="0.025" effort="50" velocity="0.1"/>
+      <limit lower="0.0" upper="0.025" effort="200" velocity="0.1"/>
     	<axis xyz="0.0 -1.0 0.0"/>
   </joint>
   <link name='finger1'>
       <inertial>
-      <origin xyz="0 0 0.02" rpy="0 0 0"/>
-      <mass value="0.0001" />
-      <inertia  ixx="0.0" ixy="0.0"  ixz="0.0"  iyy="0.0"  iyz="0.0"  izz="0.0" />
+      <origin xyz="0 0 0.0" rpy="0 0 0"/>
+      <mass value="0.01" />
+      <inertia  ixx="0.0001" ixy="0.0"  ixz="0.0"  iyy="0.0001"  iyz="0.0"  izz="0.0001" />
       </inertial>
       <visual name='visual'>
@@ -542,5 +542,5 @@
       <origin xyz="0 0 0.02" rpy="0 0 0"/>
         <geometry>
-        <box size="0.01 0.01 0.04" />
+        <box size="0.01 0.01 0.04"/>
         </geometry>
       </collision>
@@ -550,12 +550,12 @@
       <parent link="hand"/>
       <child link="finger2"/>
-      <limit lower="0.0" upper="0.025" effort="50" velocity="0.1"/>
+      <limit lower="0.0" upper="0.025" effort="200" velocity="0.1"/>
     	<axis xyz="0.0 1.0 0.0"/>
   </joint>
   <link name='finger2'>
       <inertial>
-      <origin xyz="0 0 0.02" rpy="0 0 0"/>
-      <mass value="0.0001" />
-      <inertia  ixx="0.0" ixy="0.0"  ixz="0.0"  iyy="0.0"  iyz="0.0"  izz="0.0" />
+      <origin xyz="0 0 0.0" rpy="0 0 0"/>
+      <mass value="0.01" />
+      <inertia  ixx="0.0001" ixy="0.0"  ixz="0.0"  iyy="0.0001"  iyz="0.0"  izz="0.0001" />
       </inertial>
       <visual name='visual'>
