Commit message: Add stl files for the car, and build up the whole car. The control of the roller haven't been done yet.

File: tel_map/urdf/sakura.gazebo.xacro (robot description, xacro)
@@ -1,7 +1,13 @@
-<?xml version="1.0"?>
-<robot name="SAKURA" xmlns:xacro="http://ros.org/wiki/xacro">
+<?xml version="1.0" ?>
+<robot name="sakura_setting" xmlns:xacro="http://ros.org/wiki/xacro">
   <xacro:arg name="laser_visual" default="false"/>
   <xacro:arg name="camera_visual" default="false"/>
   <xacro:arg name="imu_visual"   default="false"/>
+  <gazebo>
+    <plugin name="gazebo_ros_control" filename="libgazebo_ros_control.so">
+      <legacyModeNS>true</legacyModeNS>
+      <robotNamespace>/sakura</robotNamespace>
+    </plugin>
+  </gazebo>
   <gazebo reference="base_link">
     <material>Gazebo/DarkGrey</material>
@@ -64,10 +70,10 @@
   </gazebo>
   <gazebo>
-    <plugin name="mc_steering" filename="libgazebo_ros_planar_move.so">
+    <plugin name="mc_steering" filename="libgazebo_ros_mc_move.so">
       <commandTopic>cmd_vel</commandTopic>
       <odometryTopic>odom</odometryTopic>
       <odometryFrame>odom</odometryFrame>
       <odometryRate>30.0</odometryRate>
-      <robotBaseFrame>base_footprint</robotBaseFrame>
+      <robotBaseFrame>base_link</robotBaseFrame>
       <publishTf>true</publishTf>
     </plugin>
@@ -164,3 +170,133 @@
     </sensor>
   </gazebo>
+  <transmission name="t_plate_joint">
+      <type>transmission_interface/SimpleTransmission</type>
+      <joint name="plate_joint">
+        <hardwareInterface>hardware_interface/EffortJointInterface</hardwareInterface>
+      </joint>
+      <actuator name="plate_joint">
+        <mechanicalReduction>1</mechanicalReduction>
+        <hardwareInterface>hardware_interface/EffortJointInterface</hardwareInterface>
+      </actuator>
+   </transmission>
+  <transmission name="t_j1_joint">
+      <type>transmission_interface/SimpleTransmission</type>
+      <joint name="j1_joint">
+        <hardwareInterface>hardware_interface/EffortJointInterface</hardwareInterface>
+      </joint>
+      <actuator name="j1_joint">
+        <mechanicalReduction>1</mechanicalReduction>
+        <hardwareInterface>hardware_interface/EffortJointInterface</hardwareInterface>
+      </actuator>
+   </transmission>
+  <transmission name="t_j2_joint">
+      <type>transmission_interface/SimpleTransmission</type>
+      <joint name="j2_joint">
+        <hardwareInterface>hardware_interface/EffortJointInterface</hardwareInterface>
+      </joint>
+      <actuator name="j2_joint">
+        <mechanicalReduction>1</mechanicalReduction>
+        <hardwareInterface>hardware_interface/EffortJointInterface</hardwareInterface>
+      </actuator>
+   </transmission>
+  <transmission name="t_j3_joint">
+      <type>transmission_interface/SimpleTransmission</type>
+      <joint name="j3_joint">
+        <hardwareInterface>hardware_interface/EffortJointInterface</hardwareInterface>
+      </joint>
+      <actuator name="j3_joint">
+        <mechanicalReduction>1</mechanicalReduction>
+        <hardwareInterface>hardware_interface/EffortJointInterface</hardwareInterface>
+      </actuator>
+   </transmission>
+  <transmission name="t_j4_joint">
+      <type>transmission_interface/SimpleTransmission</type>
+      <joint name="j4_joint">
+        <hardwareInterface>hardware_interface/EffortJointInterface</hardwareInterface>
+      </joint>
+      <actuator name="j4_joint">
+        <mechanicalReduction>1</mechanicalReduction>
+        <hardwareInterface>hardware_interface/EffortJointInterface</hardwareInterface>
+      </actuator>
+   </transmission>
+  <transmission name="f1_joint">
+    <type>transmission_interface/SimpleTransmission</type>
+    <joint name="f1_joint">
+      <hardwareInterface>hardware_interface/EffortJointInterface</hardwareInterface>
+    </joint>
+    <actuator name="f1_joint">
+      <mechanicalReduction>1</mechanicalReduction>
+      <hardwareInterface>hardware_interface/EffortJointInterface</hardwareInterface>
+    </actuator>
+  </transmission>
+  <transmission name="f2_joint">
+    <type>transmission_interface/SimpleTransmission</type>
+    <joint name="f2_joint">
+      <hardwareInterface>hardware_interface/EffortJointInterface</hardwareInterface>
+    </joint>
+    <actuator name="f2_joint">
+      <mechanicalReduction>1</mechanicalReduction>
+      <hardwareInterface>hardware_interface/EffortJointInterface</hardwareInterface>
+    </actuator>
+  </transmission>
+  <transmission name="rot_joint">
+      <type>transmission_interface/SimpleTransmission</type>
+      <joint name="rot_joint">
+        <hardwareInterface>hardware_interface/EffortJointInterface</hardwareInterface>
+      </joint>
+      <actuator name="rot_joint">
+        <mechanicalReduction>1</mechanicalReduction>
+        <hardwareInterface>hardware_interface/EffortJointInterface</hardwareInterface>
+      </actuator>
+   </transmission>
+  <transmission name="cam_yaw_joint">
+      <type>transmission_interface/SimpleTransmission</type>
+      <joint name="cam_yaw_joint">
+        <hardwareInterface>hardware_interface/EffortJointInterface</hardwareInterface>
+      </joint>
+      <actuator name="cam_yaw_joint">
+        <mechanicalReduction>1</mechanicalReduction>
+        <hardwareInterface>hardware_interface/EffortJointInterface</hardwareInterface>
+      </actuator>
+   </transmission>
+  <transmission name="shovel_joint">
+      <type>transmission_interface/SimpleTransmission</type>
+      <joint name="shovel_joint">
+        <hardwareInterface>hardware_interface/EffortJointInterface</hardwareInterface>
+      </joint>
+      <actuator name="shovel_joint">
+        <mechanicalReduction>1</mechanicalReduction>
+        <hardwareInterface>hardware_interface/EffortJointInterface</hardwareInterface>
+      </actuator>
+   </transmission>
+  <transmission name="roller_arm_joint">
+      <type>transmission_interface/SimpleTransmission</type>
+      <joint name="roller_arm_joint">
+        <hardwareInterface>hardware_interface/EffortJointInterface</hardwareInterface>
+      </joint>
+      <actuator name="roller_arm_joint">
+        <mechanicalReduction>1</mechanicalReduction>
+        <hardwareInterface>hardware_interface/EffortJointInterface</hardwareInterface>
+      </actuator>
+   </transmission>
+  <transmission name="roller_arm_slider">
+      <type>transmission_interface/SimpleTransmission</type>
+      <joint name="roller_arm_slider">
+        <hardwareInterface>hardware_interface/EffortJointInterface</hardwareInterface>
+      </joint>
+      <actuator name="roller_arm_slider">
+        <mechanicalReduction>1</mechanicalReduction>
+        <hardwareInterface>hardware_interface/EffortJointInterface</hardwareInterface>
+      </actuator>
+   </transmission>
+  <transmission name="roller_joint">
+      <type>transmission_interface/SimpleTransmission</type>
+      <joint name="roller_joint">
+        <hardwareInterface>hardware_interface/EffortJointInterface</hardwareInterface>
+      </joint>
+      <actuator name="roller_joint">
+        <mechanicalReduction>1</mechanicalReduction>
+        <hardwareInterface>hardware_interface/EffortJointInterface</hardwareInterface>
+      </actuator>
+   </transmission>
 </robot>

File: tel_map/urdf/sakura.urdf.xacro (robot description, xacro)
@@ -6,31 +6,145 @@
   <joint name="base_joint" type="fixed">
     <parent link="base_footprint"/>
-    <child link="base_link"/>
+    <child link="mc_base"/>
     <origin xyz="0.0 0.0 0.0" rpy="0 0 0"/>
   </joint>
-  <link name="base_link">
+  <link name="mc_base">
     <visual>
       <origin xyz="0.3 0.135 0.015" rpy="1.57079 0 -1.57079"/>
       <geometry>
-        <mesh filename="package://tel_map/meshes/bases/sakura_base.stl" scale="0.001 0.001 0.001"/>
+        <mesh filename="package://tel_map/meshes/bases/main.stl" scale="0.001 0.001 0.001"/>
       </geometry>
       <material name="light_black"/>
     </visual>
     <collision>
-      <origin xyz="0.0 0 0.15" rpy="0 0 0"/>
-      <geometry>
-        <box size="0.280 0.280 0.20"/>
-      </geometry>
-    </collision>
-    <inertial>
-      <origin xyz="0 0 0" rpy="0 0 0"/>
-      <mass value="8.2573504e-01"/>
-      <inertia ixx="2.2124416e-03" ixy="-1.2294101e-05" ixz="3.4938785e-05"
-               iyy="2.1193702e-03" iyz="-5.0120904e-06"
-               izz="2.0064271e-03" />
-    </inertial>
-  </link>
+      <origin xyz="0.0 0 0.07" rpy="0 0 0"/>
+      <geometry>
+        <box size="0.280 0.280 0.05"/>
+      </geometry>
+    </collision>
+    <inertial>
+      <origin xyz="0 0 0" rpy="0 0 0"/>
+      <mass value="200.0"/>
+      <inertia ixx="0.1" ixy="-0.001" ixz="0.0001"
+               iyy="0.1" iyz="0.001"
+               izz="0.1" />
+    </inertial>
+  </link>
+  <!--Shovel-->>
+  <joint name="shovel_joint" type="revolute">
+    <parent link="base_footprint"/>
+    <child link="shovel_link"/>
+    <origin xyz="-0.077 0.0 0.105" rpy="0 0 0"/>
+    <limit lower="-0.1" upper="3.0416" effort="50" velocity="7.5"/>
+    <axis xyz="0.0 1.0 0.0"/>
+  </joint>
+  <link name="shovel_link">
+    <visual>
+      <origin xyz="0.028 0.14 0.375" rpy="3.14159 0 -1.57079"/>
+      <geometry>
+        <mesh filename="package://tel_map/meshes/bases/shovel.stl" scale="0.001 0.001 0.001"/>
+      </geometry>
+      <material name="light_black"/>
+    </visual>
+    <collision  name="shovel_collision1">
+      <origin xyz="-0.15 0 -0.065" rpy="0 -0.16 0"/>
+      <geometry>
+        <box size="0.09 0.24 0.002"/>
+      </geometry>
+    </collision>
+    <collision name="shovel_collision2">
+      <origin xyz="-0.1 0 -0.035" rpy="0 -0.95 0"/>
+      <geometry>
+        <box size="0.05 0.24 0.002"/>
+      </geometry>
+    </collision>
+    <inertial>
+      <origin xyz="-0.1 0 0" />
+      <mass value="0.1" />
+      <inertia ixx="1.1175580e-05" ixy="-4.2369783e-11" ixz="-5.9381719e-09"
+               iyy="1.1192413e-05" iyz="-1.4400107e-11"
+               izz="2.0712558e-05" />
+      </inertial>
+  </link>
+  <!--roller-->>
+  <joint name="roller_arm_joint" type="revolute">
+    <parent link="base_footprint"/>
+    <child link="roller_arm_a_link"/>
+    <origin xyz="-0.069 0.0 0.083" rpy="0 0 0"/>
+    <limit lower="-2.0" upper="1.0" effort="50" velocity="7.5"/>
+    <axis xyz="0.0 1.0 0.0"/>
+  </joint>
+  <link name="roller_arm_a_link">
+    <visual>
+      <origin xyz="-0.02 0.335 -0.005" rpy="1.57079 0 0"/>
+      <geometry>
+        <mesh filename="package://tel_map/meshes/bases/roller_arm_a.stl" scale="0.001 0.001 0.001"/>
+      </geometry>
+      <material name="light_black"/>
+    </visual>
+    <inertial>
+      <origin xyz="0.0 0 0.1" />
+      <mass value="0.1" />
+      <inertia ixx="0.005" ixy="0.00005" ixz="0.00005"
+               iyy="0.005" iyz="0.00005"
+               izz="0.005" />
+    </inertial>
+  </link>
+   <joint name="roller_arm_slider" type="prismatic">
+    <parent link="roller_arm_a_link"/>
+    <child link="roller_arm_b_link"/>
+    <origin xyz="0.0 0.0 0.0" rpy="0 0 0"/>
+    <limit lower="0.0" upper="0.16" effort="250.0" velocity="0.15"/>
+    <axis xyz="0.0 0.0 1.0"/>
+    <safety_controller k_velocity="70" k_position="50" soft_lower_limit="-10.0" soft_upper_limit="10.0" />
+  </joint>
+  <link name="roller_arm_b_link">
+    <visual>
+      <origin xyz="-0.014 0.335 0.01" rpy="1.571 0 0"/>
+      <geometry>
+        <mesh filename="package://tel_map/meshes/bases/roller_arm_b.stl" scale="0.001 0.001 0.001"/>
+      </geometry>
+      <material name="light_black"/>
+    </visual>
+    <inertial>
+      <origin xyz="0.0 0 0.1" />
+      <mass value="0.05" />
+      <inertia ixx="0.005" ixy="0.00005" ixz="0.00005"
+               iyy="0.005" iyz="0.00005"
+               izz="0.005" />
+    </inertial>
+  </link>
+  <joint name="roller_joint" type="continuous">
+    <parent link="roller_arm_b_link"/>
+    <child link="roller_link"/>
+    <origin xyz="0.0 0.0 0.212" rpy="0 0 0"/>
+    <limit effort="50" velocity="7.5"/>
+    <axis xyz="0.0 1.0 0.0"/>
+  </joint>
+  <link name="roller_link">
+    <visual>
+      <origin xyz="-0.0223 -0.135 -0.022" rpy="0 0 0"/>
+      <geometry>
+        <mesh filename="package://tel_map/meshes/bases/roller.stl" scale="0.001 0.001 0.001"/>
+      </geometry>
+      <material name="light_black"/>
+    </visual>
+    <collision>
+      <origin xyz="0 0 0" rpy="1.571 0 0"/>
+      <geometry>
+        <cylinder length="0.24" radius="0.022"/>
+      </geometry>
+    </collision>
+    <inertial>
+      <origin xyz="-0.0 0 0" />
+      <mass value="0.02" />
+      <inertia ixx="1.1175580e-05" ixy="0.0" ixz="0.0"
+               iyy="1.1192413e-05" iyz="0.0"
+               izz="2.0712558e-05" />
+    </inertial>
+  </link>
+<!--wheels-->
   <joint name="wheel_left_joint" type="continuous">
-    <parent link="base_link"/>
+    <parent link="mc_base"/>
     <child link="wheel_left_link"/>
     <origin xyz="0.11 0.1 0.03" rpy="-1.57079 0 0"/>
@@ -60,5 +174,5 @@
   </link>
   <joint name="wheel_right_joint" type="continuous">
-    <parent link="base_link"/>
+    <parent link="mc_base"/>
     <child link="wheel_right_link"/>
     <origin xyz="0.11 -0.1 0.03" rpy="-1.57079 0 0"/>
@@ -88,5 +202,5 @@
   </link>
   <joint name="wheel_bleft_joint" type="continuous">
-    <parent link="base_link"/>
+    <parent link="mc_base"/>
     <child link="wheel_bleft_link"/>
     <origin xyz="-0.11 0.1 0.03" rpy="-1.57079 0 0"/>
@@ -116,5 +230,5 @@
   </link>
   <joint name="wheel_bright_joint" type="continuous">
-    <parent link="base_link"/>
+    <parent link="mc_base"/>
     <child link="wheel_bright_link"/>
     <origin xyz="-0.11 -0.1 0.03" rpy="-1.57079 0 0"/>
@@ -143,29 +257,19 @@
       </inertial>
   </link>
-  <joint name="imu_joint" type="fixed">
-    <parent link="base_link"/>
-    <child link="imu_link"/>
-    <origin xyz="-0.032 0 0.068" rpy="0 0 0"/>
-  </joint>
-  <link name="imu_link"/>
-  <joint name="scan_joint" type="fixed">
-    <parent link="base_link"/>
-    <child link="base_scan"/>
-    <origin xyz="0.05 0 0.28" rpy="0 0 0"/>
-  </joint>
-  <link name="base_scan">
-    <visual>
-      <origin xyz="0 0 0.0" rpy="0 0 0"/>
-      <geometry>
-        <mesh filename="package://tel_map/meshes/sensors/lds.stl" scale="0.001 0.001 0.001"/>
-      </geometry>
-      <material name="dark"/>
-    </visual>
-    <collision>
-      <origin xyz="0.015 0 -0.0065" rpy="0 0 0"/>
-      <geometry>
-        <cylinder length="0.0315" radius="0.055"/>
-      </geometry>
-    </collision>
+  <joint name="rot_joint" type="revolute">
+    <parent link="base_footprint"/>
+    <child link="rot_link"/>
+    <origin xyz="0.067 -0.12 0.278" rpy="0 0 0"/>
+    <limit lower="0.0" upper="4.7124" effort="120" velocity="7.5"/>
+    <axis xyz="0.0 1.0 0.0"/>
+  </joint>
+  <link name="rot_link">
+    <visual>
+    <origin xyz="-0.243 0.238 0.0" rpy="-1.28 0 -1.57079"/>
+      <geometry>
+        <mesh filename="package://tel_map/meshes/bases/rot.stl" scale="0.001 0.001 0.001"/>
+      </geometry>
+      <material name="light_black"/>
+    </visual>
     <inertial>
       <mass value="0.114" />
@@ -176,26 +280,65 @@
     </inertial>
   </link>
-  <joint name="camera_joint" type="fixed">
-    <origin xyz="0.040 -0.011 0.16" rpy="0 0.0 0"/>
-    <parent link="base_link"/>
-    <child link="camera_link"/>
-  </joint>
+  <joint name="imu_joint" type="fixed">
+    <parent link="mc_base"/>
+    <child link="imu_link"/>
+    <origin xyz="-0.032 0 0.068" rpy="0 0 0"/>
+  </joint>
+  <link name="imu_link"/>
+  <joint name="scan_joint" type="fixed">
+    <parent link="rot_link"/>
+    <child link="base_scan"/>
+    <origin xyz="0.05 0 0.0" rpy="0 0 0"/>
+  </joint>
+  <link name="base_scan">
+    <visual>
+      <origin xyz="-0.038 0.118 0.025" rpy="0 0 0"/>
+      <geometry>
+        <mesh filename="package://tel_map/meshes/sensors/lds.stl" scale="0.001 0.001 0.001"/>
+      </geometry>
+      <material name="dark"/>
+    </visual>
+    <collision>
+      <origin xyz="-0.038 0.118 0.025" rpy="0 0 0"/>
+      <geometry>
+        <cylinder length="0.0315" radius="0.055"/>
+      </geometry>
+    </collision>
+    <inertial>
+      <mass value="0.114" />
+      <origin xyz="-0.038 0.118 0.025" rpy="0 0 0"/>
+      <inertia ixx="0.001" ixy="0.0" ixz="0.0"
+               iyy="0.001" iyz="0.0"
+               izz="0.001" />
+    </inertial>
+  </link>
+<joint name="cam_yaw_joint" type="revolute">
+      <origin xyz="0.0 0.118 -0.05" rpy="0 0 0"/>
+      <parent link="rot_link"/>
+      <child link="camera_link"/>
+      <limit lower="-1.57" upper="1.57" effort="50" velocity="7.5"/>
+    	<axis xyz="0.0 0.0 1.0"/>
+      <calibration rising="0.0"/>
+      <dynamics damping="0.0" friction="0.0"/>
+      <safety_controller k_velocity="80" k_position="50" soft_lower_limit="-5.0" soft_upper_limit="5.0" />
+    </joint>
   <link name="camera_link">
-    <collision>
-      <origin xyz="0.005 0.011 0.013" rpy="0 0 0"/>
-      <geometry>
-        <box size="0.015 0.030 0.027"/>
-      </geometry>
-    </collision>
-    <visual>
-      <origin xyz="0.005 0.011 0.013" rpy="0 0 0"/>
+    <visual>
+      <origin xyz="0.0 0.0 0.0" rpy="0 0 0"/>
       <geometry>
         <box size="0.02 0.08 0.02"/>
       </geometry>
-      <material name="light_black"/>
-    </visual>
+      <material name="blue"/>
+    </visual>
+    <inertial>
+      <mass value="0.114" />
+      <origin xyz="-0.0 0.0 0.0" rpy="0 0 0"/>
+      <inertia ixx="0.001" ixy="0.0" ixz="0.0"
+               iyy="0.001" iyz="0.0"
+               izz="0.001" />
+    </inertial>
   </link>
   <joint name="camera_rgb_joint" type="fixed">
-    <origin xyz="0.003 0.011 0.009" rpy="0 0 0"/>
+    <origin xyz="0.0 0.0 0.0" rpy="0 0 0"/>
     <parent link="camera_link"/>
     <child link="camera_rgb_frame"/>
@@ -208,3 +351,218 @@
   </joint>
   <link name="camera_rgb_optical_frame"/>
+<joint name="arm_base_joint" type="fixed">
+    <origin xyz="0.12 -0.10 0.075" rpy="0 0 0"/>
+    <parent link="base_footprint"/>
+    <child link="arm_base"/>
+    </joint>
+  <link name='arm_base'>
+      <inertial>
+      <origin xyz="0 0 0" />
+      <mass value="0.001" />
+      <inertia  ixx="0.0" ixy="0.0"  ixz="0.0"  iyy="0.0"  iyz="0.0"  izz="0.0" />
+      </inertial>
+      <visual name='visual'>
+      <origin xyz="0 0 0"/>
+        <geometry>
+        <box size="0.04 0.015 0.025" />
+        </geometry>
+      </visual>
+      <collision name='collision'>
+      <origin xyz="0 0 0"/>
+        <geometry>
+        <box size="0.04 0.015 0.025" />
+        </geometry>
+      </collision>
+    </link>
+<joint name="plate_joint" type="revolute">
+    <origin xyz="0 0 0.064" rpy="0 0 0"/>
+      <parent link="arm_base"/>
+      <child link="plate"/>
+      <limit lower="-1.57" upper="1.57" effort="50" velocity="7.5"/>
+    	<axis xyz="0.0 0.0 1.0"/>
+      <calibration rising="0.0"/>
+      <dynamics damping="0.0" friction="0.0"/>
+      <safety_controller k_velocity="80" k_position="50" soft_lower_limit="-5.0" soft_upper_limit="5.0" />
+    </joint>
+<link name='plate'>
+      <inertial>
+      <origin xyz="0 0 0.0" />
+      <mass value="0.001" />
+      <inertia  ixx="0.0" ixy="0.0"  ixz="0.0"  iyy="0.0"  iyz="0.0"  izz="0.0" />
+      </inertial>
+      <visual name='visual'>
+      <origin xyz="0 0 0.0"/>
+        <geometry>
+        <box size="0.04 0.04 0.025" />
+        </geometry>
+      </visual>
+      <collision name='collision'>
+      <origin xyz="0 0 0.0"/>
+        <geometry>
+        <box size="0.04 0.04 0.025" />
+        </geometry>
+      </collision>
+    </link>
+<joint name="j1_joint" type="revolute">
+    <origin xyz="0 0 0.0" rpy="0 0 0"/>
+      <parent link="plate"/>
+      <child link="link2"/>
+      <limit lower="-1.57" upper="1.57" effort="50" velocity="7.5"/>
+    	<axis xyz="0.0 1.0 0.0"/>
+      <calibration rising="0.0"/>
+      <dynamics damping="0.0" friction="0.0"/>
+      <safety_controller k_velocity="80" k_position="50" soft_lower_limit="-5.0" soft_upper_limit="5.0" />
+    </joint>
+<link name='link2'>
+      <inertial>
+      <origin xyz="0 0 0.05215" />
+      <mass value="0.001" />
+      <inertia  ixx="0.0" ixy="0.0"  ixz="0.0"  iyy="0.0"  iyz="0.0"  izz="0.0" />
+      </inertial>
+      <visual name='visual'>
+      <origin xyz="0 0 0.05215"/>
+        <geometry>
+        <box size="0.025 0.0564 0.1043" />
+        </geometry>
+      </visual>
+      <collision name='collision'>
+      <origin xyz="0 0 0.05215"/>
+        <geometry>
+        <box size="0.025 0.0564 0.1043" />
+        </geometry>
+      </collision>
+    </link>
+<joint name="j2_joint" type="revolute">
+    <origin xyz="0 0 0.1043" rpy="0 0 0.0"/>
+      <parent link="link2"/>
+      <child link="link3"/>
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
Commit message: add the third challenge add the roller control

File: tel_map/urdf/sakura.gazebo.xacro (robot description, xacro)
@@ -1,5 +1,5 @@
 <?xml version="1.0" ?>
 <robot name="sakura_setting" xmlns:xacro="http://ros.org/wiki/xacro">
-  <xacro:arg name="laser_visual" default="false"/>
+  <xacro:arg name="laser_visual" default="true"/>
   <xacro:arg name="camera_visual" default="false"/>
   <xacro:arg name="imu_visual"   default="false"/>
@@ -77,4 +77,5 @@
       <robotBaseFrame>base_link</robotBaseFrame>
       <publishTf>true</publishTf>
+      <roller>roller_joint</roller>
     </plugin>
   </gazebo>
@@ -106,8 +107,8 @@
     </plugin>
   </gazebo>
-  <gazebo reference="base_scan">
+  <gazebo reference="scaner_link">
     <material>Gazebo/FlatBlack</material>
     <sensor type="ray" name="lds_lfcd_sensor">
-      <pose>0 0 0 0 0 0</pose>
+      <pose>0.0 0.0 0.0 0 0 0</pose>
       <visualize>$(arg laser_visual)</visualize>
       <update_rate>5</update_rate>

File: tel_map/urdf/sakura.urdf.xacro (robot description, xacro)
@@ -119,5 +119,5 @@
     <child link="roller_link"/>
     <origin xyz="0.0 0.0 0.212" rpy="0 0 0"/>
-    <limit effort="50" velocity="7.5"/>
+    <limit effort="500" velocity="20000.0"/>
     <axis xyz="0.0 1.0 0.0"/>
   </joint>
@@ -313,4 +313,10 @@
     </inertial>
   </link>
+  <joint name="scaner_joint" type="fixed">
+    <parent link="base_scan"/>
+    <child link="scaner_link"/>
+    <origin xyz="-0.038 0.118 0.025" rpy="0 0 0"/>
+  </joint>
+  <link name="scaner_link"/>
 <joint name="cam_yaw_joint" type="revolute">
       <origin xyz="0.0 0.118 -0.05" rpy="0 0 0"/>
