Commit message: Fix the gripper again.

File: tel_map/urdf/sakura.gazebo.xacro (robot description, xacro)
@@ -50,4 +50,39 @@
     <minDepth>0.001</minDepth>
     <maxVel>0.1</maxVel>
+    <fdir1>1 0 0</fdir1>
+    <material>Gazebo/FlatBlack</material>
+  </gazebo>
+  <gazebo reference="plate">
+    <material>Gazebo/FlatBlack</material>
+  </gazebo>
+  <gazebo reference="link2">
+    <material>Gazebo/FlatBlack</material>
+  </gazebo>
+  <gazebo reference="link3">
+    <material>Gazebo/FlatBlack</material>
+  </gazebo>
+  <gazebo reference="link4">
+    <material>Gazebo/FlatBlack</material>
+  </gazebo>
+  <gazebo reference="hand">
+    <material>Gazebo/FlatBlack</material>
+  </gazebo>
+  <gazebo reference="finger1">
+    <mu1>88.0</mu1>
+    <mu2>88.0</mu2>
+    <kp>500000.0</kp>
+    <kd>10.0</kd>
+    <minDepth>0.002</minDepth>
+    <maxVel>0.0</maxVel>
+    <fdir1>1 0 0</fdir1>
+    <material>Gazebo/FlatBlack</material>
+  </gazebo>
+  <gazebo reference="finger2">
+    <mu1>88.0</mu1>
+    <mu2>88.0</mu2>
+    <kp>500000.0</kp>
+    <kd>10.0</kd>
+    <minDepth>0.002</minDepth>
+    <maxVel>0.0</maxVel>
     <fdir1>1 0 0</fdir1>
     <material>Gazebo/FlatBlack</material>

File: tel_map/urdf/sakura.urdf.xacro (robot description, xacro)
@@ -157,5 +157,4 @@
         <cylinder length="0.018" radius="0.03"/>
       </geometry>
-      <material name="dark"/>
     </visual>
     <collision>
@@ -460,4 +459,5 @@
         <box size="0.025 0.0564 0.091" />
         </geometry>
+      <material name="light_black"/>
       </visual>
       <collision name='collision'>
@@ -524,5 +524,5 @@
       <parent link="hand"/>
       <child link="finger1"/>
-      <limit lower="0.0" upper="0.025" effort="200" velocity="0.1"/>
+      <limit lower="0.0" upper="0.025" effort="30" velocity="0.1"/>
     	<axis xyz="0.0 -1.0 0.0"/>
   </joint>
@@ -530,6 +530,6 @@
       <inertial>
       <origin xyz="0 0 0.0" rpy="0 0 0"/>
-      <mass value="0.01" />
-      <inertia  ixx="0.0001" ixy="0.0"  ixz="0.0"  iyy="0.0001"  iyz="0.0"  izz="0.0001" />
+      <mass value="0.05" />
+      <inertia  ixx="0.0001" ixy="0.00000001"  ixz="0.00000001"  iyy="0.0001"  iyz="0.00000001"  izz="0.0001" />
       </inertial>
       <visual name='visual'>
@@ -544,5 +544,41 @@
         <box size="0.01 0.01 0.04"/>
         </geometry>
-      </collision>
+        <surface>
+          <friction>
+            <ode>
+              <mu>100000</mu>
+              <mu2>100000</mu2>
+            </ode>
+          </friction>
+        </surface>
+      </collision>
+      <!--collision>
+      <origin xyz="0 -0.002 0.035" rpy="0 0 0"/>
+        <geometry>
+          <sphere radius="0.005"/>
+        </geometry>
+        <surface>
+          <friction>
+            <ode>
+              <mu>1000</mu>
+              <mu2>500</mu2>
+            </ode>
+          </friction>
+        </surface>
+      </collision>
+      <collision>
+      <origin xyz="0 -0.002 0.025" rpy="0 0 0"/>
+        <geometry>
+          <sphere radius="0.005"/>
+        </geometry>
+        <surface>
+          <friction>
+            <ode>
+              <mu>1000</mu>
+              <mu2>500</mu2>
+            </ode>
+          </friction>
+        </surface>
+      </collision-->
   </link>
   <joint name="f2_joint" type="prismatic">
@@ -550,5 +586,5 @@
       <parent link="hand"/>
       <child link="finger2"/>
-      <limit lower="0.0" upper="0.025" effort="200" velocity="0.1"/>
+      <limit lower="0.0" upper="0.025" effort="30" velocity="0.1"/>
     	<axis xyz="0.0 1.0 0.0"/>
   </joint>
@@ -556,6 +592,6 @@
       <inertial>
       <origin xyz="0 0 0.0" rpy="0 0 0"/>
-      <mass value="0.01" />
-      <inertia  ixx="0.0001" ixy="0.0"  ixz="0.0"  iyy="0.0001"  iyz="0.0"  izz="0.0001" />
+      <mass value="0.05" />
+      <inertia  ixx="0.0001" ixy="0.00000001"  ixz="0.00000001"  iyy="0.0001"  iyz="0.00000001"  izz="0.0001" />
       </inertial>
       <visual name='visual'>
@@ -568,7 +604,43 @@
       <origin xyz="0 0 0.02" rpy="0 0 0"/>
         <geometry>
-        <box size="0.01 0.01 0.04" />
-        </geometry>
-      </collision>
+          <box size="0.01 0.01 0.04" />
+        </geometry>
+        <surface>
+          <friction>
+            <ode>
+              <mu>100000</mu>
+              <mu2>100000</mu2>
+            </ode>
+          </friction>
+        </surface>
+      </collision>
+      <!---collision>
+      <origin xyz="0 0.002 0.035" rpy="0 0 0"/>
+        <geometry>
+          <sphere radius="0.005"/>
+        </geometry>
+        <surface>
+          <friction>
+            <ode>
+              <mu>1000</mu>
+              <mu2>500</mu2>
+            </ode>
+          </friction>
+        </surface>
+      </collision>
+      <collision>
+      <origin xyz="0 0.002 0.025" rpy="0 0 0"/>
+        <geometry>
+          <sphere radius="0.005"/>
+        </geometry>
+        <surface>
+          <friction>
+            <ode>
+              <mu>1000</mu>
+              <mu2>500</mu2>
+            </ode>
+          </friction>
+        </surface>
+      </collision-->
   </link>
 </robot>

Commit message: This is the final version of the map. Don't mass it up again, game holders!

File: tel_map/urdf/sakura.gazebo.xacro (robot description, xacro)
@@ -14,6 +14,6 @@
   </gazebo>
   <gazebo reference="wheel_left_link">
-    <mu1>0.1</mu1>
-    <mu2>0.1</mu2>
+    <mu1>0.0</mu1>
+    <mu2>0.0</mu2>
     <kp>500000.0</kp>
     <kd>10.0</kd>
@@ -24,6 +24,6 @@
   </gazebo>
   <gazebo reference="wheel_right_link">
-    <mu1>0.1</mu1>
-    <mu2>0.1</mu2>
+    <mu1>0.0</mu1>
+    <mu2>0.0</mu2>
     <kp>500000.0</kp>
     <kd>10.0</kd>
@@ -34,6 +34,6 @@
   </gazebo>
   <gazebo reference="wheel_bleft_link">
-    <mu1>0.1</mu1>
-    <mu2>0.1</mu2>
+    <mu1>0.0</mu1>
+    <mu2>0.0</mu2>
     <kp>500000.0</kp>
     <kd>10.0</kd>
@@ -44,6 +44,6 @@
   </gazebo>
   <gazebo reference="wheel_bright_link">
-    <mu1>0.1</mu1>
-    <mu2>0.1</mu2>
+    <mu1>0.0</mu1>
+    <mu2>0.0</mu2>
     <kp>500000.0</kp>
     <kd>10.0</kd>
@@ -106,5 +106,5 @@
   <gazebo>
     <plugin name="mc_steering" filename="$(find tel_map)/lib/libgazebo_ros_mc_move.so">
-      <commandTopic>cmd_vel</commandTopic>
+      <commandTopic>/sakura/cmd_vel</commandTopic>
       <odometryTopic>odom</odometryTopic>
       <odometryFrame>odom</odometryFrame>
@@ -181,5 +181,5 @@
           <horizontal_fov>0.8</horizontal_fov>
           <image>
-              <width>360</width>
+              <width>320</width>
               <height>240</height>
               <format>R8G8B8</format>

File: tel_map/urdf/sakura.urdf.xacro (robot description, xacro)
@@ -473,5 +473,5 @@
       <child link="link4"/>
       <limit lower="-1.57" upper="1.57" effort="50" velocity="7.5"/>
-    	<axis xyz="0.0 1.0 0.0"/>
+    	<axis xyz="0.0 -1.0 0.0"/>
       <calibration rising="0.0"/>
       <dynamics damping="0.0" friction="0.0"/>
